Commit message: Add custom mesh files

File: src/silver/description/gazebo_control.xacro (robot description, xacro)
@@ -2,6 +2,4 @@
 <robot xmlns:xacro="http://www.ros.org/wiki/xacro">
   <gazebo>
-    <!-- <plugin filename="gz_ros2_control-system" name="gz_ros2_control::GazeboSimROS2ControlPlugin"> -->
-    <!-- <plugin filename="libgazebo_ros2_control.so" name="gazebo_ros2_control"> -->
     <plugin filename="libgz_ros2_control-system.so" name="gz_ros2_control::GazeboSimROS2ControlPlugin">
       <robot_param>robot_description</robot_param>

File: src/silver/description/silver.xacro (robot description, xacro)
@@ -27,9 +27,8 @@
     <link name="body_link">
         <visual>
-            <origin xyz="0.0 0.0 0.0" rpy="0.0 0.0 0.0"/>
+            <origin xyz="0.0 0.0 0.0" rpy="1.57 0.0 1.57"/>
             <geometry>
-                <box size="${body_link_x_dim} ${body_link_y_dim} ${body_link_z_dim}"/>
+                <mesh filename="$(find silver)/models/silver2/meshes/SILVER2_Body_Simplified.fbx" scale="0.45 0.45 0.55"/>
             </geometry>
-            <material name="blue"/>
         </visual>
         <collision>
@@ -43,7 +42,4 @@
         </xacro:inertial_box>
     </link>
-    <gazebo reference="body_link">
-      <material>Gazebo/Blue</material>
-    </gazebo>
     <xacro:leg suffix="0" reflect="1" side='right' Ox="0.275" Oy="-0.2" Oz="-0.15"/>
     <xacro:leg suffix="1" reflect="1" side='right' Ox="0.0" Oy="-0.2" Oz="-0.15"/>

File: src/silver/description/silver_constants.xacro (robot description, xacro)
@@ -14,4 +14,7 @@
     <xacro:property name="coxa_link_Oy" value="-0.05" /> <!-- m -->
     <xacro:property name="coxa_link_Oz" value="-0.05" /> <!-- m -->
+    <xacro:property name="coxa_link_visual_Ox" value="0.03" /> <!-- m -->
+    <xacro:property name="coxa_link_visual_Oy" value="-0.075" /> <!-- m -->
+    <xacro:property name="coxa_link_visual_Oz" value="0.075" /> <!-- m -->
     <xacro:property name="coxa_link_Ry" value="1.57" /> <!-- rad -->
     <xacro:property name="coxa_link_length" value="0.1" /> <!-- m -->
@@ -21,8 +24,11 @@
     <xacro:property name="femur_joint_Oy" value="-0.05" /> <!-- m -->
     <xacro:property name="femur_joint_Oz" value="-0.05" /> <!-- m -->
-    <xacro:property name="femur_joint_Ry" value="-1.57" /> <!-- rad -->
+    <xacro:property name="femur_joint_Ry" value="-1.57" /> <!-- -1.57 rad -->
     <xacro:property name="femur_link_Ox" value="0.0" /> <!-- m -->
     <xacro:property name="femur_link_Oy" value="-0.15" /> <!-- m -->
     <xacro:property name="femur_link_Oz" value="-0.03" /> <!-- m -->
+    <xacro:property name="femur_link_visual_Ox" value="0.01" /> <!-- m -->
+    <xacro:property name="femur_link_visual_Oy" value="0.0" /> <!-- m -->
+    <xacro:property name="femur_link_visual_Oz" value="0.02" /> <!-- m -->
     <xacro:property name="femur_link_dx" value="0.03" /> <!-- m -->
     <xacro:property name="femur_link_dy" value="0.3" /> <!-- m -->
@@ -36,4 +42,7 @@
     <xacro:property name="tibia_link_Oy" value="-0.15" /> <!-- m -->
     <xacro:property name="tibia_link_Oz" value="0.0" /> <!-- m -->
+    <xacro:property name="tibia_link_visual_Ox" value="0.0" /> <!-- m -->
+    <xacro:property name="tibia_link_visual_Oy" value="-0.0" /> <!-- m -->
+    <xacro:property name="tibia_link_visual_Oz" value="0.0" /> <!-- m -->
     <xacro:property name="tibia_link_dx" value="0.03" /> <!-- m -->
     <xacro:property name="tibia_link_dy" value="0.27" /> <!-- m -->

File: src/silver/description/silver_leg.xacro (robot description, xacro)
@@ -14,16 +14,14 @@
             <limit effort="250.0" velocity="10.0" lower="-3.14" upper="3.14" />
             <axis xyz="0 0 1"/>
-            <!--dynamics damping="10.0" friction="10.0"/-->
         </joint>
         <link name="coxa_link_${suffix}">
             <visual>
-                <origin xyz="${reflect*coxa_link_Ox} ${coxa_link_Oy} ${coxa_link_Oz}" rpy="0.0 ${coxa_link_Ry} 0.0"/>
+                <origin xyz="${reflect*coxa_link_visual_Ox} ${coxa_link_visual_Oy} ${coxa_link_visual_Oz}" rpy="1.57 0.0 0.0"/>
                 <geometry>
-                    <cylinder length="${coxa_link_length}" radius="${coxa_link_radius}"/>
+                    <mesh filename="$(find silver)/models/silver2/meshes/SILVER2_Coxa_Simplified.fbx" scale="0.45 0.45 0.45"/>
                 </geometry>
-                <material name="red"/>
             </visual>
             <collision>
-                <origin xyz="${reflect*coxa_link_Ox} ${coxa_link_Oy} ${coxa_link_Oz}" rpy="0.0 ${coxa_link_Ry} 0.0"/>
+                <origin xyz="${reflect*coxa_link_Ox} ${coxa_link_Oy} ${coxa_link_Oz}" rpy="0.0 ${coxa_link_Ry} 0.0"/> <!--dynamics damping="10.0" friction="10.0"/-->
                 <geometry>
                     <cylinder length="${coxa_link_length}" radius="${coxa_link_radius}"/>
@@ -34,7 +32,4 @@
             </xacro:inertial_cylinder>
         </link>
-        <gazebo reference="coxa_link_${suffix}">
-            <material>Gazebo/Blue</material>
-        </gazebo>
         <!-- FEMUR JOINT AND LINK-->
         <joint name="femur_joint_${suffix}" type="revolute">
@@ -47,9 +42,8 @@
         <link name="femur_link_${suffix}">
             <visual>
-                <origin xyz="${femur_link_Ox} ${femur_link_Oy} ${reflect*femur_link_Oz}" rpy="0.0 0.0 0.0"/>
+                <origin xyz="${femur_link_visual_Ox} ${femur_link_visual_Oy} ${reflect*femur_link_visual_Oz}" rpy="0.0 0.0 0.0"/>
                 <geometry>
-                    <box size="${femur_link_dx} ${femur_link_dy} ${femur_link_dz}"/>
+                    <mesh filename="$(find silver)/models/silver2/meshes/SILVER2_Femur_Simplified.fbx" scale="0.5 0.5 0.5"/>
                 </geometry>
-                <material name="orange"/>
             </visual>
             <collision>
@@ -63,7 +57,4 @@
             </xacro:inertial_box>
         </link>
-        <gazebo reference="femur_link_${suffix}">
-            <material>Gazebo/Orange</material>
-        </gazebo>
         <!-- TIBIA JOINT AND LINK -->
         <joint name="tibia_joint_${suffix}" type="revolute">
@@ -76,9 +67,8 @@
         <link name="tibia_link_${suffix}">
             <visual>
-                <origin xyz="${tibia_link_Ox} ${tibia_link_Oy} ${tibia_link_Oz}" rpy="0.0 0.0 0.0"/>
+                <origin xyz="${tibia_link_visual_Ox} ${tibia_link_visual_Oy} ${tibia_link_visual_Oz}" rpy="0.0 0.0 0.0"/>
                 <geometry>
-                    <box size="${tibia_link_dx} ${tibia_link_dy} ${tibia_link_dz}"/>
+                    <mesh filename="$(find silver)/models/silver2/meshes/SILVER2_Tibia_Simplified.fbx" scale="0.5 0.45 0.5"/>
                 </geometry>
-                <material name="black"/>
             </visual>
             <collision>
@@ -92,34 +82,4 @@
             </xacro:inertial_box>
         </link>
-        <gazebo reference="tibia_link_${suffix}">
-            <material>Gazebo/Black</material>
-        </gazebo>
-        <!-- FOOT JOINT AND LINK -->
-        <joint name="foot_joint_${suffix}" type="fixed">
-            <origin xyz="${foot_joint_Ox} ${foot_joint_Oy} ${foot_joint_Oz}" rpy="0.0 0.0 0.0"/>
-            <parent link="tibia_link_${suffix}"/>
-            <child link="foot_link_${suffix}"/>
-        </joint>
-        <link name="foot_link_${suffix}">
-            <visual>
-                <origin xyz="${foot_link_Ox} ${foot_link_Oy} ${foot_link_Oz}" rpy="0.0 0.0 0.0"/>
-                <geometry>
-                    <sphere radius="${foot_radius}"/>
-                </geometry>
-                <material name="white"/>
-            </visual>
-            <collision>
-                <origin xyz="${foot_link_Ox} ${foot_link_Oy} ${foot_link_Oz}" rpy="0.0 0.0 0.0"/>
-                <geometry>
-                    <sphere radius="${foot_radius}"/>
-                </geometry>
-            </collision>
-            <xacro:inertial_sphere mass="${foot_mass}" radius="${foot_radius}">
-                <origin xyz="${foot_link_Ox} ${foot_link_Oy} ${foot_link_Oz}" rpy="0.0 0.0 0.0"/>
-            </xacro:inertial_sphere>
-        </link>
-        <gazebo reference="foot_link_${suffix}">
-            <material>Gazebo/White</material>
-        </gazebo>
     </xacro:macro>
 </robot>

Commit message: Include Hydrodynamics

File: src/silver/description/gazebo_control.xacro (robot description, xacro)
@@ -7,4 +7,32 @@
       <parameters>$(find silver)/config/silver_controllers.yaml</parameters>
     </plugin>
+    <!-- Hydrodynamics plugin
+    <plugin
+      filename="gz-sim-hydrodynamics-system"
+      name="gz::sim::systems::Hydrodynamics">
+      <link_name>base_link</link_name>
+      <!
+      <xDotU>-0.04876161</xDotU>
+      <yDotV>-1.26324739</yDotV>
+      <zDotW>-1.26324739</zDotW>
+      <kDotP>0</kDotP>
+      <mDotQ>-0.3346</mDotQ>
+      <nDotR>-0.3346</nDotR>
+        Note about added mass: SDFormat also supports added mass natively.
+        Until we deprecate the added mass parameters of this plugin, do not set the added mass parameters in both places,
+        choose one (either in this plugin or under <inertial> of your link).
+      <xUabsU>73.8</xUabsU>
+      <xU>0</xU>
+      <yVabsV>84.9</yVabsV>
+      <yV>0</yV>
+      <zWabsW>882.7</zWabsW>
+      <zW>0</zW>
+      <kPabsP>-40.0</kPabsP>
+      <kP>0</kP>
+      <mQabsQ>-60.0</mQabsQ>
+      <mQ>0</mQ>
+      <nRabsR>-50.0</nRabsR>
+      <nR>0</nR>
+    </plugin>-->
   </gazebo>
 </robot>

Commit message: Fix SILVER2 Hydrodynamics

File: src/silver/description/gazebo_control.xacro (robot description, xacro)
@@ -7,32 +7,26 @@
       <parameters>$(find silver)/config/silver_controllers.yaml</parameters>
     </plugin>
-    <!-- Hydrodynamics plugin
+     <!-- Hydrodynamics plugin -->
     <plugin
       filename="gz-sim-hydrodynamics-system"
       name="gz::sim::systems::Hydrodynamics">
+      <!-- Link this plugin is attached to -->
       <link_name>base_link</link_name>
-      <!
-      <xDotU>-0.04876161</xDotU>
-      <yDotV>-1.26324739</yDotV>
-      <zDotW>-1.26324739</zDotW>
-      <kDotP>0</kDotP>
-      <mDotQ>-0.3346</mDotQ>
-      <nDotR>-0.3346</nDotR>
-        Note about added mass: SDFormat also supports added mass natively.
-        Until we deprecate the added mass parameters of this plugin, do not set the added mass parameters in both places,
-        choose one (either in this plugin or under <inertial> of your link).
-      <xUabsU>73.8</xUabsU>
+      <!-- Linear Damping Coefficients -->
       <xU>0</xU>
-      <yVabsV>84.9</yVabsV>
       <yV>0</yV>
-      <zWabsW>882.7</zWabsW>
       <zW>0</zW>
-      <kPabsP>-40.0</kPabsP>
+      <!-- Quadratic Damping Coefficients (Halved to not crash the sim)-->
+      <xUabsU>35.0</xUabsU> <!-- 73.8 -->
+      <yVabsV>42.0</yVabsV> <!-- 84.9 -->
+      <zWabsW>440.0</zWabsW> <!-- 882.7 -->
+      <!-- Rotational Damping Coefficients -->
       <kP>0</kP>
-      <mQabsQ>-60.0</mQabsQ>
       <mQ>0</mQ>
-      <nRabsR>-50.0</nRabsR>
       <nR>0</nR>
-    </plugin>-->
+      <kPabsP>40.0</kPabsP>
+      <mQabsQ>60.0</mQabsQ>
+      <nRabsR>50.0</nRabsR>
+    </plugin>
   </gazebo>
 </robot>

Commit message: Update physics and terrain

File: src/silver/description/gazebo_control.xacro (robot description, xacro)
@@ -7,25 +7,20 @@
       <parameters>$(find silver)/config/silver_controllers.yaml</parameters>
     </plugin>
-     <!-- Hydrodynamics plugin -->
     <plugin
       filename="gz-sim-hydrodynamics-system"
       name="gz::sim::systems::Hydrodynamics">
-      <!-- Link this plugin is attached to -->
       <link_name>base_link</link_name>
-      <!-- Linear Damping Coefficients -->
-      <xU>0</xU>
-      <yV>0</yV>
-      <zW>0</zW>
-      <!-- Quadratic Damping Coefficients (Halved to not crash the sim)-->
-      <xUabsU>35.0</xUabsU> <!-- 73.8 -->
-      <yVabsV>42.0</yVabsV> <!-- 84.9 -->
-      <zWabsW>440.0</zWabsW> <!-- 882.7 -->
-      <!-- Rotational Damping Coefficients -->
-      <kP>0</kP>
-      <mQ>0</mQ>
-      <nR>0</nR>
-      <kPabsP>40.0</kPabsP>
-      <mQabsQ>60.0</mQabsQ>
-      <nRabsR>50.0</nRabsR>
+        <xU>0.296</xU>
+        <yV>0.296</yV>
+        <zW>0.592</zW>
+        <kP>0.06</kP>
+        <mQ>0.06</mQ>
+        <nR>0.08</nR>
+        <xUabsU>2.952</xUabsU>
+        <yVabsV>2.952</yVabsV>
+        <zWabsW>5.904</zWabsW>
+        <kPabsP>0.6</kPabsP>
+        <mQabsQ>0.6</mQabsQ>
+        <nRabsR>0.8</nRabsR>
     </plugin>
   </gazebo>

File: src/silver/description/silver.xacro (robot description, xacro)
@@ -20,9 +20,4 @@
     <link name = "base_link"></link>
     <!-- BODY JOINT AND LINK -->
-    <joint name="body_joint" type="fixed">
-        <origin xyz="0.0 0.0 0.4" rpy="0.0 0.0 0.0"/>
-        <parent link="base_link"/>
-        <child link="body_link"/>
-    </joint>
     <link name="body_link">
         <visual>
@@ -42,4 +37,9 @@
         </xacro:inertial_box>
     </link>
+    <joint name="body_joint" type="fixed">
+        <origin xyz="0.0 0.0 0.4" rpy="0.0 0.0 0.0"/>
+        <parent link="base_link"/>
+        <child link="body_link"/>
+    </joint>
     <xacro:leg suffix="0" reflect="1" side='right' Ox="0.275" Oy="-0.2" Oz="-0.15"/>
     <xacro:leg suffix="1" reflect="1" side='right' Ox="0.0" Oy="-0.2" Oz="-0.15"/>

File: src/silver/description/silver_constants.xacro (robot description, xacro)
@@ -2,7 +2,7 @@
 <robot xmlns:xacro="http://www.ros.org/wiki/xacro" >
     <!-- Constant parameters -->
-    <xacro:property name="body_link_mass" value="140.0" /> <!-- Kg -->
+    <xacro:property name="body_link_mass" value="50.0" /> <!-- 140 Kg -->
     <xacro:property name="body_link_height" value="1.0" /> <!-- m -->
-    <xacro:property name="body_link_x_dim" value="0.55" /> <!-- m -->
+    <xacro:property name="body_link_x_dim" value="0.4" /> <!-- m -->
     <xacro:property name="body_link_y_dim" value="0.4" /> <!-- m -->
     <xacro:property name="body_link_z_dim" value="0.3" /> <!-- m -->
