Commit message: Update Visuals

File: src/silver/description/silver.xacro (robot description, xacro)
@@ -27,7 +27,7 @@
     <link name="body_link">
         <visual>
-            <origin xyz="0.0 0.0 0.0" rpy="1.57 0.0 1.57"/>
+            <origin xyz="0.05 0.0 0.0" rpy="1.57 0.0 1.57"/>
             <geometry>
-                <mesh filename="$(find silver)/models/silver2/meshes/SILVER2_Body_Simplified.fbx" scale="0.45 0.45 0.55"/>
+                <mesh filename="file://$(find silver)/models/silver2/meshes/SILVER2_Body_Simplified.fbx" scale="0.35 0.4 0.45"/>
             </geometry>
         </visual>

File: src/silver/description/silver_constants.xacro (robot description, xacro)
@@ -14,7 +14,7 @@
     <xacro:property name="coxa_link_Oy" value="-0.05" /> <!-- m -->
     <xacro:property name="coxa_link_Oz" value="-0.05" /> <!-- m -->
-    <xacro:property name="coxa_link_visual_Ox" value="0.03" /> <!-- m -->
-    <xacro:property name="coxa_link_visual_Oy" value="-0.075" /> <!-- m -->
-    <xacro:property name="coxa_link_visual_Oz" value="0.075" /> <!-- m -->
+    <xacro:property name="coxa_link_visual_Ox" value="0.0" /> <!-- 0.03m -->
+    <xacro:property name="coxa_link_visual_Oy" value="0.0" /> <!-- -0.075 m -->
+    <xacro:property name="coxa_link_visual_Oz" value="0.0" /> <!-- 0.075m -->
     <xacro:property name="coxa_link_Ry" value="1.57" /> <!-- rad -->
     <xacro:property name="coxa_link_length" value="0.1" /> <!-- m -->
@@ -28,7 +28,7 @@
     <xacro:property name="femur_link_Oy" value="-0.15" /> <!-- m -->
     <xacro:property name="femur_link_Oz" value="-0.03" /> <!-- m -->
-    <xacro:property name="femur_link_visual_Ox" value="0.01" /> <!-- m -->
+    <xacro:property name="femur_link_visual_Ox" value="0.0" /> <!-- 0.01m -->
     <xacro:property name="femur_link_visual_Oy" value="0.0" /> <!-- m -->
-    <xacro:property name="femur_link_visual_Oz" value="0.02" /> <!-- m -->
+    <xacro:property name="femur_link_visual_Oz" value="0.0" /> <!-- 0.02m -->
     <xacro:property name="femur_link_dx" value="0.03" /> <!-- m -->
     <xacro:property name="femur_link_dy" value="0.3" /> <!-- m -->
@@ -43,5 +43,5 @@
     <xacro:property name="tibia_link_Oz" value="0.0" /> <!-- m -->
     <xacro:property name="tibia_link_visual_Ox" value="0.0" /> <!-- m -->
-    <xacro:property name="tibia_link_visual_Oy" value="-0.0" /> <!-- m -->
+    <xacro:property name="tibia_link_visual_Oy" value="0.01" /> <!-- m -->
     <xacro:property name="tibia_link_visual_Oz" value="0.0" /> <!-- m -->
     <xacro:property name="tibia_link_dx" value="0.03" /> <!-- m -->

File: src/silver/description/silver_leg.xacro (robot description, xacro)
@@ -19,5 +19,5 @@
                 <origin xyz="${reflect*coxa_link_visual_Ox} ${coxa_link_visual_Oy} ${coxa_link_visual_Oz}" rpy="1.57 0.0 0.0"/>
                 <geometry>
-                    <mesh filename="$(find silver)/models/silver2/meshes/SILVER2_Coxa_Simplified.fbx" scale="0.45 0.45 0.45"/>
+                    <mesh filename="file://$(find silver)/models/silver2/meshes/SILVER2_Coxa_Simplified.fbx" scale="0.45 0.45 0.45"/>
                 </geometry>
             </visual>
@@ -44,5 +44,5 @@
                 <origin xyz="${femur_link_visual_Ox} ${femur_link_visual_Oy} ${reflect*femur_link_visual_Oz}" rpy="0.0 0.0 0.0"/>
                 <geometry>
-                    <mesh filename="$(find silver)/models/silver2/meshes/SILVER2_Femur_Simplified.fbx" scale="0.5 0.5 0.5"/>
+                    <mesh filename="file://$(find silver)/models/silver2/meshes/SILVER2_Femur_Simplified.fbx" scale="0.5 0.5 0.5"/>
                 </geometry>
             </visual>
@@ -69,5 +69,5 @@
                 <origin xyz="${tibia_link_visual_Ox} ${tibia_link_visual_Oy} ${tibia_link_visual_Oz}" rpy="0.0 0.0 0.0"/>
                 <geometry>
-                    <mesh filename="$(find silver)/models/silver2/meshes/SILVER2_Tibia_Simplified.fbx" scale="0.5 0.45 0.5"/>
+                    <mesh filename="file://$(find silver)/models/silver2/meshes/SILVER2_Tibia_Simplified.fbx" scale="0.5 0.45 0.5"/>
                 </geometry>
             </visual>

Commit message: Update Coordinates + Visuals

File: src/silver/description/silver.xacro (robot description, xacro)
@@ -22,5 +22,5 @@
     <link name="body_link">
         <visual>
-            <origin xyz="0.05 0.0 0.0" rpy="1.57 0.0 1.57"/>
+            <origin xyz="0.05 0.0 0.0" rpy="1.57 0.0 -1.57"/>
             <geometry>
                 <mesh filename="file://$(find silver)/models/silver2/meshes/SILVER2_Body_Simplified.fbx" scale="0.35 0.4 0.45"/>
